Commit message: Adjust collision coordinates and dimensions

File: phylax_description/urdf/phylax.urdf.xacro (robot description, xacro)
@@ -19,6 +19,7 @@
         <link name="base_link">
                 <collision>
+                        <origin xyz="0 0 0.02" rpy="0 0 0"/>
                         <geometry>
-                                <box size="0.39 0.188 0.19"/>
+                                <box size="0.37 0.165 0.08"/>
                         </geometry>
                 </collision>
@@ -42,4 +43,10 @@
                         </geometry>
                 </visual>
+                <collision>
+                        <origin xyz="0 0 -0.015" rpy="0 0 0"/>
+                        <geometry>
+                                <box size="0.38 0.12 0.034"/>
+                        </geometry>
+                </collision>
         </link>
         <joint name="base_link_joint" type="fixed">
@@ -53,5 +60,5 @@
                 <origin xyz="0.0 0.0 0.06" rpy="0 0 0"/>
         </joint>
-        <xacro:macro name="wheel" params="pos side xyz rpy xyzi rpyi">
+        <xacro:macro name="wheel" params="pos side xyz rpy xyzi rpyi cy">
                 <link name="${pos}_${side}_wheel">
                         <visual>
@@ -62,7 +69,7 @@
                         </visual>
                         <collision>
-                                <origin xyz="0 0 0" rpy="0 0 0"/>
+                                <origin xyz="0 ${cy} 0" rpy="${PI/2} 0 0"/>
                                 <geometry>
-                                        <cylinder radius="0.06" length="0.06"/>
+                                        <cylinder radius="0.06" length="0.062"/>
                                 </geometry>
                         </collision>
@@ -96,10 +103,10 @@
                 </transmission>
         </xacro:macro>
-        <xacro:wheel pos="front" side="left"  xyz="-0.15 -0.08 -0.02" rpy="${PI/2} 0 0" xyzi="0.15 0.08 0.0" rpyi="0 0 0" />
-        <xacro:wheel pos="front" side="right" xyz="-0.15 0.08 0.02" rpy="${-PI/2} 0 0" xyzi="0.15 -0.08 0.0" rpyi="0 0 0" />
-        <xacro:wheel pos="center" side="left"  xyz="-0.15 -0.08 -0.02" rpy="${PI/2} 0 0"  xyzi="0.0 0.08 0.0" rpyi="0 0 0"/>
-        <xacro:wheel pos="center" side="right" xyz="-0.15 0.08 0.02" rpy="${-PI/2} 0 0"  xyzi="0.0 -0.08 0.0" rpyi="0 0 0"/>
-        <xacro:wheel pos="rear" side="left"  xyz="-0.15 -0.08 -0.02" rpy="${PI/2} 0 0"  xyzi="-0.15 0.08 0.0" rpyi="0 0 0"/>
-        <xacro:wheel pos="rear" side="right" xyz="-0.15 0.08 0.02" rpy="${-PI/2} 0 0" xyzi="-0.15 -0.08 0.0" rpyi="0 0 0"/>
+        <xacro:wheel pos="front" side="left"  xyz="-0.15 -0.08 -0.02" rpy="${PI/2} 0 0" xyzi="0.15 0.08 0.0" rpyi="0 0 0" cy="0.038"/>
+        <xacro:wheel pos="front" side="right" xyz="-0.15 0.08 0.02" rpy="${-PI/2} 0 0" xyzi="0.15 -0.08 0.0" rpyi="0 0 0" cy="-0.038"/>
+        <xacro:wheel pos="center" side="left"  xyz="-0.15 -0.08 -0.02" rpy="${PI/2} 0 0"  xyzi="0.0 0.08 0.0" rpyi="0 0 0" cy="0.038"/>
+        <xacro:wheel pos="center" side="right" xyz="-0.15 0.08 0.02" rpy="${-PI/2} 0 0"  xyzi="0.0 -0.08 0.0" rpyi="0 0 0" cy="-0.038"/>
+        <xacro:wheel pos="rear" side="left"  xyz="-0.15 -0.08 -0.02" rpy="${PI/2} 0 0"  xyzi="-0.15 0.08 0.0" rpyi="0 0 0" cy="0.038"/>
+        <xacro:wheel pos="rear" side="right" xyz="-0.15 0.08 0.02" rpy="${-PI/2} 0 0" xyzi="-0.15 -0.08 0.0" rpyi="0 0 0" cy="-0.038"/>
         <gazebo>
                 <plugin name="gazebo_ros_control" filename="libgazebo_ros_control.so">

Commit message: Fix urdf file

File: phylax_description/urdf/phylax.urdf.xacro (robot description, xacro)
@@ -1,10 +1,5 @@
 <?xml version="1.0"?>
 <robot name="Phylax" xmlns:xacro="http://www.ros.org/wiki/xacro">
-<material name="Black">
-   <color rgba="0.0 0.0 0.0 1.0"/>
-</material>
-<material name="White">
-   <color rgba="1.0 1.0 1.0 1.0"/>
-</material>
+<xacro:include filename="$(find phylax_description)/urdf/phylax.gazebo.xacro" />
 <xacro:property name="deg_to_rad" value="0.017453"/>
 <xacro:property name="PI" value="3.14"/>
@@ -35,5 +30,5 @@
    <transmission name="${joint_name}_trans">
     <type>transmission_interface/SimpleTransmission</type>
-     <joint name="${joint_name}">      <geometry>
+     <joint name="${joint_name}">
        <hardwareInterface>PositionJointInterface</hardwareInterface>
      </joint>
@@ -65,8 +60,7 @@
     </geometry>
   </visual>
-  <collision>/>
+  <collision>/><origin rpy="${PI/2} 0 0" xyz="0 0 -0.018"/>
     <geometry>
-    <origin rpy="${PI/2} 0 0" xyz="0 0 -0.018"
-       <mesh filename="package://phylax_description/meshes/wild_thumper_6wd_chassis.stl" scale="0.001 0.001 0.001"/>
+      <mesh filename="package://phylax_description/meshes/wild_thumper_6wd_chassis.stl" scale="0.001 0.001 0.001"/>
     </geometry>
   </collision>
@@ -78,7 +72,4 @@
     <origin xyz="0 0 ${wheel_radius}" rpy="0 0 0"/>
   </joint>
- <gazebo reference="chassis_link">
-    <turnGravityOff>false</turnGravityOff>
-  </gazebo>
   <link name="top_chassis">
       <visual>
@@ -89,12 +80,12 @@
       </visual>
   </link>
-    <joint name="top_chassis_joint" type="fixed">
-        <parent link="chassis_link"/>
-        <child link="top_chassis"/>
-        <origin rpy="0 0 0" xyz="0.0 0.0 0.058"/>
-        <axis xyz="0 1 0"/>
-        <limit effort="100" velocity="100"/>
-        <dynamics damping="0.0" friction="0.0"/>
-    </joint>
+  <joint name="top_chassis_joint" type="fixed">
+    <parent link="chassis_link"/>
+    <child link="top_chassis"/>
+    <origin rpy="0 0 0" xyz="0.0 0.0 0.058"/>
+    <axis xyz="0 1 0"/>
+    <limit effort="100" velocity="100"/>
+    <dynamics damping="0.0" friction="0.0"/>
+  </joint>
 <xacro:macro name="wheel" params="pos side xyz xyzi cy">
   <link name="${pos}_${side}_wheel">
@@ -146,9 +137,3 @@
 <xacro:wheel pos="rear" side="left" xyz="-0.023 -${chassis_width/2-0.01} 0.068" xyzi="-0.150 ${chassis_width/2} 0" cy="0.036"/>
 <xacro:wheel pos="rear" side="right" xyz="-0.023 -${chassis_width-0.02} 0.068" xyzi="-0.150 -${chassis_width/2} 0" cy="-0.036"/>
-<!-- ros_control plugin-->
-<gazebo>
-  <plugin name="gazebo_ros_control" filename= "libgazebo_ros_control.so">
-   <robotNamespace>/</robotNamespace>
-  </plugin>
-</gazebo>
 </robot>

Commit message: Add a link & a joint along with the necessary xacro file for the velodyne LiDAR to the phylax urdf model

File: phylax_description/urdf/phylax.urdf.xacro (robot description, xacro)
@@ -137,3 +137,24 @@
 <xacro:wheel pos="rear" side="left" xyz="-0.023 -${chassis_width/2-0.01} 0.068" xyzi="-0.150 ${chassis_width/2} 0" cy="0.036"/>
 <xacro:wheel pos="rear" side="right" xyz="-0.023 -${chassis_width-0.02} 0.068" xyzi="-0.150 -${chassis_width/2} 0" cy="-0.036"/>
+  <xacro:include filename="$(find velodyne_description)/urdf/VLP-16.urdf.xacro"/>
+  <VLP-16 parent="top_chassis" name="velodyne" topic="/velodyne_points" gpu="true">
+    <origin xyz="-0.12 0.009 0.052" rpy="0 0 0" />
+  </VLP-16>
+  <!-- Velodyne mount stuff -->
+  <link name="velodyne_mount">
+    <visual>
+      <origin xyz="0 0 0" rpy="0.0 0.0 0.0" />
+      <geometry>
+        <mesh filename="package://phylax_description/meshes/velodyne_mount.stl"/>
+      </geometry>
+      <material name="aluminum" >
+        <color rgba="0.45 0.45 0.45 1"/>
+      </material>
+    </visual>
+  </link>
+  <joint name="velodyne_mount_joint" type="fixed">
+    <parent link="velodyne_base_link" />
+    <child link="velodyne_mount" />
+    <origin xyz="0 0 0" />
+  </joint>
 </robot>

Commit message: Remove velodyne from main urdf and load an accessories urdf. Add urdf for gps alternative lidars

File: phylax_description/urdf/phylax.urdf.xacro (robot description, xacro)
@@ -1,4 +1,4 @@
 <?xml version="1.0"?>
-<robot name="Phylax" xmlns:xacro="http://www.ros.org/wiki/xacro">
+<robot name="phylax" xmlns:xacro="http://www.ros.org/wiki/xacro">
 <xacro:include filename="$(find phylax_description)/urdf/phylax.gazebo.xacro" />
 <xacro:property name="deg_to_rad" value="0.017453"/>
@@ -137,24 +137,4 @@
 <xacro:wheel pos="rear" side="left" xyz="-0.023 -${chassis_width/2-0.01} 0.068" xyzi="-0.150 ${chassis_width/2} 0" cy="0.036"/>
 <xacro:wheel pos="rear" side="right" xyz="-0.023 -${chassis_width-0.02} 0.068" xyzi="-0.150 -${chassis_width/2} 0" cy="-0.036"/>
-  <xacro:include filename="$(find velodyne_description)/urdf/VLP-16.urdf.xacro"/>
-  <VLP-16 parent="top_chassis" name="velodyne" topic="/velodyne_points" gpu="true">
-    <origin xyz="-0.12 0.009 0.052" rpy="0 0 0" />
-  </VLP-16>
-  <!-- Velodyne mount stuff -->
-  <link name="velodyne_mount">
-    <visual>
-      <origin xyz="0 0 0" rpy="0.0 0.0 0.0" />
-      <geometry>
-        <mesh filename="package://phylax_description/meshes/velodyne_mount.stl"/>
-      </geometry>
-      <material name="aluminum" >
-        <color rgba="0.45 0.45 0.45 1"/>
-      </material>
-    </visual>
-  </link>
-  <joint name="velodyne_mount_joint" type="fixed">
-    <parent link="velodyne_base_link" />
-    <child link="velodyne_mount" />
-    <origin xyz="0 0 0" />
-  </joint>
+ <xacro:include filename="$(find jackal_description)/urdf/accessories.urdf.xacro" />
 </robot>
