Commit message: Correct application references

File: phylax_description/urdf/accessories.urdf.xacro (robot description, xacro)
@@ -27,5 +27,5 @@
     </xacro:if>
     <xacro:unless value="$(optenv PHYLAX_LASER_HOKUYO 0)">
-      <xacro:include filename="$(find PHYLAX_description)/urdf/accessories/sick_lms1xx_mount.urdf.xacro" />
+      <xacro:include filename="$(find phylax_description)/urdf/accessories/sick_lms1xx_mount.urdf.xacro" />
       <sick_lms1xx_mount prefix="$(optenv PHYLAX_LASER_MOUNT front)"
                          topic="$(optenv PHYLAX_LASER_TOPIC front/scan)"/>
@@ -40,5 +40,5 @@
   <!-- If enabled, generate the upgraded Navsat payload (a Novatel Smart6). -->
   <xacro:if value="$(optenv PHYLAX_NAVSAT 0)">
-    <xacro:include filename="$(find PHYLAX_description)/urdf/accessories/novatel_smart6.urdf.xacro" />
+    <xacro:include filename="$(find phylax_description)/urdf/accessories/novatel_smart6.urdf.xacro" />
     <bridge_plate mount="$(optenv PHYLAX_NAVSAT_MOUNT rear)"
                   height="$(optenv PHYLAX_NAVSAT_HEIGHT 0.1)" />

File: phylax_description/urdf/accessories/bridge_plate.urdf.xacro (robot description, xacro)
@@ -11,5 +11,5 @@
         <origin xyz="0 0 0" rpy="1.5707 0.0 1.5707" />
         <geometry>
-          <mesh filename="package://jackal_description/meshes/bridge-plate.stl"/>
+          <mesh filename="package://phylax_description/meshes/bridge-plate.stl"/>
         </geometry>
         <material name="dark_grey" />

File: phylax_description/urdf/phylax.urdf.xacro (robot description, xacro)
@@ -137,4 +137,4 @@
 <xacro:wheel pos="rear" side="left" xyz="-0.023 -${chassis_width/2-0.01} 0.068" xyzi="-0.150 ${chassis_width/2} 0" cy="0.036"/>
 <xacro:wheel pos="rear" side="right" xyz="-0.023 -${chassis_width-0.02} 0.068" xyzi="-0.150 -${chassis_width/2} 0" cy="-0.036"/>
- <xacro:include filename="$(find jackal_description)/urdf/accessories.urdf.xacro" />
+ <xacro:include filename="$(find phylax_description)/urdf/accessories.urdf.xacro" />
 </robot>

Commit message: Fix parent for laser_mount_joint

File: phylax_description/urdf/accessories.urdf.xacro (robot description, xacro)
@@ -1,12 +1,4 @@
 <?xml version="1.0"?>
 <robot xmlns:xacro="http://www.ros.org/wiki/xacro">
-  <!--
-    As you add to this URDF, please be aware that both the robot and
-    simulation include it. You must retain compatibility with all of
-    the following launch files:
-    jackal_viz/launch/view_model.launch
-    jackal_gazebo/launch/phylax_world.launch
-    jackal_base/launch/base.launch
-  -->
   <!-- Macros to generate standoffs for offset payload mounting. -->
   <xacro:include filename="$(find phylax_description)/urdf/accessories/standoffs.urdf.xacro" />
@@ -33,5 +25,5 @@
         <origin xyz="$(optenv PHYLAX_LASER_OFFSET 0 0 0)"
                 rpy="$(optenv PHYLAX_LASER_RPY 0 0 0)" />
-        <parent link="$(optenv PHYLAX_LASER_MOUNT front)_mount" />
+        <parent link="top_chassis" />
         <child link="$(optenv PHYLAX_LASER_MOUNT front)_laser_mount" />
       </joint>

Commit message: Fix parent link in the laser_mount_joynt for the Hokuyo and center it

File: phylax_description/urdf/accessories.urdf.xacro (robot description, xacro)
@@ -12,7 +12,7 @@
                           topic="$(optenv PHYLAX_LASER_TOPIC front/scan)" />
       <joint name="$(optenv PHYLAX_LASER_MOUNT front)_laser_mount_joint" type="fixed">
-        <origin xyz="$(optenv PHYLAX_LASER_OFFSET 0.11 0 0)"
+        <origin xyz="$(optenv PHYLAX_LASER_OFFSET 0 0 0)"
                 rpy="$(optenv PHYLAX_LASER_RPY 0 0 0)" />
-        <parent link="$(optenv PHYLAX_LASER_MOUNT front)_mount" />
+        <parent link="top_chassis" />
         <child link="$(optenv PHYLAX_LASER_MOUNT front)_laser_mount" />
       </joint>

Commit message: Add VLP-16 as an optional accessory selectable by an environment variable

File: phylax_description/urdf/accessories.urdf.xacro (robot description, xacro)
@@ -30,4 +30,17 @@
     </xacro:unless>
   </xacro:if>
+  <xacro:unless value="$(optenv PHYLAX_LASER_VLP-16 0)">
+      <xacro:include filename="$(find velodyne_description)/urdf/VLP-16.urdf.xacro"/>
+      <VLP-16 parent="top_chassis" name="velodyne" topic="/velodyne_points">
+        <origin xyz="0 0 0" rpy="0 0 0" />
+      </VLP-16>
+    <joint name="$(optenv PHYLAX_LASER_MOUNT front)_laser_mount_joint" type="fixed">
+      <origin xyz="$(optenv PHYLAX_LASER_OFFSET 0 0 0)"
+              rpy="$(optenv PHYLAX_LASER_RPY 0 0 0)" />
+      <parent link="top_chassis" />
+      <child link="$(optenv PHYLAX_LASER_MOUNT front)_laser_mount" />
+    </joint>
+  </xacro:unless>
+</xacro:if>
   <!-- If enabled, generate the upgraded Navsat payload (a Novatel Smart6). -->
   <xacro:if value="$(optenv PHYLAX_NAVSAT 0)">

Commit message: Add VLP-16 support

File: phylax_description/urdf/accessories.urdf.xacro (robot description, xacro)
@@ -8,15 +8,4 @@
   <xacro:if value="$(optenv PHYLAX_LASER 0)">
     <xacro:if value="$(optenv PHYLAX_LASER_HOKUYO 0)">
-      <xacro:include filename="$(find phylax_description)/urdf/accessories/hokuyo_ust10.urdf.xacro" />
-      <hokuyo_ust10_mount prefix="$(optenv PHYLAX_LASER_MOUNT front)"
-                          topic="$(optenv PHYLAX_LASER_TOPIC front/scan)" />
-      <joint name="$(optenv PHYLAX_LASER_MOUNT front)_laser_mount_joint" type="fixed">
-        <origin xyz="$(optenv PHYLAX_LASER_OFFSET 0 0 0)"
-                rpy="$(optenv PHYLAX_LASER_RPY 0 0 0)" />
-        <parent link="top_chassis" />
-        <child link="$(optenv PHYLAX_LASER_MOUNT front)_laser_mount" />
-      </joint>
-    </xacro:if>
-    <xacro:unless value="$(optenv PHYLAX_LASER_HOKUYO 0)">
       <xacro:include filename="$(find phylax_description)/urdf/accessories/sick_lms1xx_mount.urdf.xacro" />
       <sick_lms1xx_mount prefix="$(optenv PHYLAX_LASER_MOUNT front)"
@@ -28,18 +17,11 @@
         <child link="$(optenv PHYLAX_LASER_MOUNT front)_laser_mount" />
       </joint>
-    </xacro:unless>
-  </xacro:if>
-  <xacro:unless value="$(optenv PHYLAX_LASER_VLP-16 0)">
+    </xacro:if>
+    <xacro:unless value="$(optenv PHYLAX_LASER_VELODYNE 0)">
       <xacro:include filename="$(find velodyne_description)/urdf/VLP-16.urdf.xacro"/>
       <VLP-16 parent="top_chassis" name="velodyne" topic="/velodyne_points">
         <origin xyz="0 0 0" rpy="0 0 0" />
       </VLP-16>
-    <joint name="$(optenv PHYLAX_LASER_MOUNT front)_laser_mount_joint" type="fixed">
-      <origin xyz="$(optenv PHYLAX_LASER_OFFSET 0 0 0)"
-              rpy="$(optenv PHYLAX_LASER_RPY 0 0 0)" />
-      <parent link="top_chassis" />
-      <child link="$(optenv PHYLAX_LASER_MOUNT front)_laser_mount" />
-    </joint>
-  </xacro:unless>
+    </xacro:unless>
 </xacro:if>
   <!-- If enabled, generate the upgraded Navsat payload (a Novatel Smart6). -->
